Commit message: set pelvis as base linnk

File: src/robots/g1_description/urdf/g1_29dof_rev_1_0.urdf (robot description, URDF)
Before this commit: robot g1_29dof_rev_1_0, 42 links, 41 joints
Links:
- removed link base_link
- removed link robot_center
Joints:
- removed joint base_link_to_pelvis
- removed joint robot_center_to_base_link
